File: ADCurrentDongle.kicad_pcb (KiCad board)
At the start: 4 copper layers, 35 x 74 mm, 54 parts, among them J1 EXT_SONDE1, J10 Conn_01x06, J2 EXT_SONDE2, J3 Screw_Terminal_01x04, J4 Conn_01x02, J5 BRD_EXT, J6 R_EXT, J7 Conn_01x03, J8 Conn_01x03, J9 Conn_01x03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

Commit message: adding new rev fabrication and stuff
Routing:
- net Net-(D3-Pad2): track 0.00 -> 51.8 mm, vias 0 -> 2
- net Net-(D4-Pad2): track 13.2 -> 42.5 mm, vias 0 -> 1
- net Net-(C6-Pad1): track 28.8 -> 53.9 mm, vias 0 -> 2
- net Net-(C5-Pad1): track 49.6 -> 69.8 mm, vias 2 -> 3
- net Net-(J9-Pad2): track 32.7 -> 27.6 mm, vias 1 -> 0
- net VDC: track 16.3 -> 18.5 mm, vias 8 -> 9
- net /VDC_JP: track 0.00 -> 1.43 mm
- net Net-(R10-Pad2): track 11.7 -> 12.5 mm
- net Net-(J10-Pad5): track 29.6 -> 29.8 mm, vias 1 -> 0
Other:
- outline, holes or cut-outs redrawn
- board text added: "(C) critbit 03.2022"
- board text added: "1+|1-|GND"
- board text added: "2+|2-|GND"
- board text added: "AnalogDiscoveryCurrentDongle Rev. 2.0"
- board text added: "CH1 CURR/BNC"
- board text added: "CH2 CURR/BNC"
- board text removed: "<-BNC"
- board text removed: "AnalogDiscovery CurrentDongle Rev. 1.1 (C) critbit"
- board text removed: "CURR->"
- board text removed: "G"
- board text removed: "GND"
- board text removed: "W1"
- board text removed: "W2"
