File: ADCurrentDongle.kicad_pcb (KiCad board)
At the start: 2 copper layers, 53.8 x 44 mm, 51 parts, among them J1 EXT_SONDE1, J2 EXT_SONDE2, J3 BRD_EXT, J4 Screw_Terminal_01x04, J5 Conn_01x02, J6 R_EXT, J7 Conn_01x03, U1 INA186AxDDxx, U2 INA186AxDDxx, U3 MCP6004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

Commit message: commiting WIP in hope of catching a routing bug
Parts:
- removed the JP5 at (76.1, 86.3)
- removed JP6: Jumper_2_Open, Connector_PinHeader_2.54mm:PinHeader_1x02_P2.54mm_Vertical
- removed JP7: CH2_SEL, Connector_PinHeader_2.54mm:PinHeader_1x03_P2.54mm_Vertical
- removed JP8: CH1_SEL, Connector_PinHeader_2.54mm:PinHeader_1x03_P2.54mm_Vertical
- added J10: Conn_01x06, Connector_PinHeader_2.54mm:PinHeader_1x06_P2.54mm_Vertical, F.Cu at (56.5, 56.8)
- added J7: Conn_01x03, Connector_PinHeader_2.54mm:PinHeader_1x03_P2.54mm_Vertical, F.Cu at (73.6, 97.8)
- added J8: Conn_01x03, Connector_PinHeader_2.54mm:PinHeader_1x03_P2.54mm_Vertical, F.Cu at (73.7, 72.8)
- added R18: 50, Resistor_SMD:R_0805_2012Metric, F.Cu at (59.0, 101.3)
- added SW1: CURR_LP_SEL, Button_Switch_SMD:SW_DPDT_CK_JS202011JCQN, F.Cu at (61.0, 56.0)
- added SW2: CH1_DPDT, Button_Switch_SMD:SW_DPDT_CK_JS202011JCQN, F.Cu at (66.2, 95.2)
- added SW3: CH2_DPDT, Button_Switch_SMD:SW_DPDT_CK_JS202011JCQN, F.Cu at (66.2, 70.2)
- C1, C2, C3, C4, C5, C6, C7, C8, C9: footprint Capacitor_SMD:C_0603_1608Metric_Pad1.08x0.95mm_HandSolder -> Capacitor_SMD:C_0402_1005Metric
- D3, D4: footprint LED_SMD:LED_0805_2012Metric_Pad1.15x1.40mm_HandSolder -> LED_SMD:LED_0603_1608Metric
- R10, R11, R12, R13, R14, R15, R16, R17, R4, R5, R8, R9: footprint Resistor_SMD:R_0603_1608Metric_Pad0.98x0.95mm_HandSolder -> Resistor_SMD:R_0402_1005Metric
- R19: renamed from R18; value 100 -> 50; footprint Resistor_SMD:R_0603_1608Metric_Pad0.98x0.95mm_HandSolder -> Resistor_SMD:R_0805_2012Metric
- R6: renamed from R7; footprint Resistor_SMD:R_0603_1608Metric_Pad0.98x0.95mm_HandSolder -> Resistor_SMD:R_0402_1005Metric
- R7: renamed from R6; footprint Resistor_SMD:R_0603_1608Metric_Pad0.98x0.95mm_HandSolder -> Resistor_SMD:R_0402_1005Metric
- moved J2 36.5 mm to (63.7, 82.8)
- moved R12 35.8 mm to (84.0, 54.6), turned to 180 degrees
- moved J1 34.8 mm to (63.7, 107.8)
- moved C8 34.8 mm to (84.0, 55.8), turned to 180 degrees
- moved R8 32.6 mm to (64.0, 51.6), turned to -90 degrees
- moved R15 31.3 mm to (86.1, 54.6), turned to 0 degrees
- moved C6 29.8 mm to (88.0, 64.9), turned to -90 degrees
- moved R16 29.6 mm to (87.8, 47.3)
- moved R9 29.0 mm to (64.0, 53.8), turned to 90 degrees
- moved R6 28.2 mm to (64.0, 57.8), turned to -90 degrees
- moved D1 25.9 mm to (86.0, 64.8), turned to 0 degrees
- moved R14 25.2 mm to (86.1, 55.9), turned to 180 degrees
- moved C5 25.0 mm to (82.1, 64.9), turned to -90 degrees
- moved R7 24.8 mm to (64.0, 59.9), turned to 90 degrees
- moved R17 24.1 mm to (87.8, 53.0)
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- renumbered J4 to J3, J5 to J4, J3 to J5, J7 to J9, JP9 to JP5, U5 to U4
Connections:
- net Net-(C1-Pad1) renamed /VDC_JP
- net Net-(C1-Pad2) renamed /V_OUT
- J1 pad 2: GND -> Net-(J1-Pad2)
- J2 pad 2: GND -> Net-(J2-Pad2)
- R19 pad 1: VDC -> Net-(R18-Pad2)
- U4 pad 1: (no net) -> unconnected-(U4-Pad1)
- U4 pad 10: (no net) -> unconnected-(U4-Pad10)
- U4 pad 11: (no net) -> Net-(J10-Pad4)
- U4 pad 12: (no net) -> unconnected-(U4-Pad12)
- U4 pad 13: (no net) -> Net-(J10-Pad3)
- U4 pad 14: (no net) -> unconnected-(U4-Pad14)
- U4 pad 15: (no net) -> Net-(J10-Pad2)
- U4 pad 16: (no net) -> unconnected-(U4-Pad16)
- U4 pad 17: (no net) -> unconnected-(U4-Pad17)
- U4 pad 18: (no net) -> unconnected-(U4-Pad18)
- U4 pad 24: (no net) -> unconnected-(U4-Pad24)
- U4 pad 28: GND -> Net-(SW3-Pad5)
- U4 pad 3: (no net) -> unconnected-(U4-Pad3)
- U4 pad 30: GND -> Net-(SW2-Pad5)
- U4 pad 5: (no net) -> unconnected-(U4-Pad5)
- U4 pad 6: (no net) -> unconnected-(U4-Pad6)
- U4 pad 7: (no net) -> unconnected-(U4-Pad7)
- U4 pad 8: (no net) -> unconnected-(U4-Pad8)
- U4 pad 9: (no net) -> Net-(J10-Pad5)
Routing:
- net Net-(D3-Pad2): track 75.7 -> 0.00 mm, vias 3 -> 0
- net VDC: track 79.9 -> 16.3 mm, vias 6 -> 8
- net Net-(D4-Pad2): track 67.1 -> 13.2 mm, vias 1 -> 0
- net Net-(SW3-Pad5): track 0.00 -> 35.2 mm, vias 0 -> 1
- net /V_OUT: track 31.6 -> 0.00 mm
- net /VDC_JP: track 31.3 -> 0.00 mm
- net Net-(J10-Pad5): track 0.00 -> 29.6 mm, vias 0 -> 1
- net Net-(J10-Pad2): track 0.00 -> 29.3 mm
- net Net-(J10-Pad3): track 0.00 -> 28.9 mm, vias 0 -> 1
- net Net-(J10-Pad4): track 0.00 -> 28.7 mm, vias 0 -> 1
- net Net-(J9-Pad2): track 9.31 -> 32.7 mm, vias 0 -> 1
- net Net-(J2-Pad1): track 44.5 -> 21.2 mm
- net Net-(R8-Pad2): track 25.1 -> 3.13 mm
- net Net-(J2-Pad2): track 0.00 -> 21.9 mm, vias 0 -> 1
- net Net-(J1-Pad2): track 0.00 -> 21.6 mm, vias 0 -> 1
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- added copper zone on In1.Cu, net GND
- added copper zone on In2.Cu, net VDC
- removed copper zone on B.Cu, net GND
- removed copper zone on F.Cu, net VDC
Other:
- board size 53.8 x 44 mm -> 35 x 74 mm
- copper layers 2 -> 4
- net class Default removed

Commit message: pre order commit
Parts:
- removed J10: Conn_01x06, Connector_PinHeader_2.54mm:PinHeader_1x06_P2.54mm_Vertical
- added D5: LED, LED_SMD:LED_0603_1608Metric, F.Cu at (82.9, 42.8)
- added R20: 3k3, Resistor_SMD:R_0402_1005Metric, F.Cu at (78.8, 52.7)
- added SW4: CH1_DPDT, Button_Switch_SMD:SW_DPDT_CK_JS202011JCQN, F.Cu at (57.5, 107.5)
- J4: footprint Connector_PinHeader_2.54mm:PinHeader_1x02_P2.54mm_Horizontal -> Connector_PinHeader_2.54mm:PinHeader_1x02_P2.54mm_Vertical
- J9: value Conn_01x03 -> Conn_01x10; footprint Connector_PinHeader_2.54mm:PinHeader_1x03_P2.54mm_Vertical -> Connector_PinHeader_2.54mm:PinHeader_1x10_P2.54mm_Vertical
- moved J9 53.3 mm to (89.5, 66.2), turned to 180 degrees
- moved JP7 41.2 mm to (72.2, 63.9), turned to -90 degrees
- moved R19 39.6 mm to (70.2, 66.8), turned to 0 degrees
- moved R18 35.4 mm to (66.8, 66.8), turned to 0 degrees
- moved R16 9.70 mm to (79.8, 52.7)
- moved R17 7.03 mm to (80.8, 52.7)
- moved D2 6.82 mm to (76.6, 56.1), turned to 90 degrees
- moved J5 6.26 mm to (79.3, 46.1)
- moved J4 6.26 mm to (76.8, 43.6)
- moved R10 6.18 mm to (74.8, 63.6), turned to -90 degrees
- moved J3 5.25 mm to (72.2, 45.7)
- moved C1 5.19 mm to (75.9, 53.2)
- moved D3 5.05 mm to (83.0, 46.2), turned to 180 degrees
- moved D4 4.83 mm to (83.0, 51.2), turned to 180 degrees
- moved SW3 4.70 mm to (56.5, 54.6)
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- renumbered JP5 to JP7, R7 to R6, R6 to R7, SW2 to SW1, SW3 to SW2, SW1 to SW3
Connections:
- net Net-(C5-Pad1) renamed /CMEAS_A
- net Net-(C6-Pad1) renamed /CMEAS_B
- net Net-(D3-Pad2) renamed /CMEAS_B_CLIP
- net Net-(J1-Pad1) renamed /CH1_INP
- net Net-(J1-Pad2) renamed /CH1_INM
- net Net-(J2-Pad1) renamed /CH2_INP
- net Net-(J2-Pad2) renamed /CH2_INM
- D4 pad 2: Net-(D4-Pad2) -> /CMEAS_A_CLIP
- J9 pad 1: Net-(J9-Pad1) -> GND
- J9 pad 2: Net-(J9-Pad2) -> /WAV_GEN1
- J9 pad 3: GND -> /WAV_GEN2
- U3 pad 14: Net-(D4-Pad2) -> /CMEAS_A_CLIP
- U4 pad 1: unconnected-(U4-Pad1) -> /CMEAS_A_CLIP
- U4 pad 11: Net-(J10-Pad4) -> unconnected-(U4-Pad11)
- U4 pad 13: Net-(J10-Pad3) -> unconnected-(U4-Pad13)
- U4 pad 15: Net-(J10-Pad2) -> /CH1_DIO
- U4 pad 16: unconnected-(U4-Pad16) -> /CH2_DIO
- U4 pad 21: Net-(J9-Pad1) -> /WAV_GEN1
- U4 pad 22: Net-(J9-Pad2) -> /WAV_GEN2
- U4 pad 3: unconnected-(U4-Pad3) -> /DIO6
- U4 pad 4: Net-(D4-Pad2) -> /DIO14
- U4 pad 5: unconnected-(U4-Pad5) -> /DIO5
- U4 pad 6: unconnected-(U4-Pad6) -> /DIO13
- U4 pad 8: unconnected-(U4-Pad8) -> /DIO12
- U4 pad 9: Net-(J10-Pad5) -> unconnected-(U4-Pad9)
Routing:
- net /CMEAS_B_CLIP: track 0.00 -> 67.1 mm, vias 0 -> 3
- net /CMEAS_A_CLIP: track 0.00 -> 51.3 mm, vias 0 -> 3
- net /WAV_GEN1: track 0.00 -> 50.1 mm, vias 0 -> 1
- net /WAV_GEN2: track 0.00 -> 49.9 mm, vias 0 -> 1
- net /DIO6: track 0.00 -> 43.5 mm, vias 0 -> 1
- net /DIO14: track 0.00 -> 40.3 mm, vias 0 -> 1
- net /DIO12: track 0.00 -> 40.2 mm, vias 0 -> 1
- net /DIO13: track 0.00 -> 39.9 mm, vias 0 -> 1
- net /DIO5: track 0.00 -> 39.5 mm, vias 0 -> 1
- net Net-(J9-Pad2): track 32.7 -> 0.00 mm, vias 1 -> 0
- net /CH1_DIO: track 0.00 -> 32.0 mm
- net /CH2_DIO: track 0.00 -> 31.1 mm, vias 0 -> 1
- net Net-(J10-Pad5): track 29.6 -> 0.00 mm, vias 1 -> 0
- net Net-(J10-Pad2): track 29.3 -> 0.00 mm
- net Net-(J10-Pad3): track 28.9 -> 0.00 mm, vias 1 -> 0
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Other:
- board size 35 x 74 mm -> 37 x 74 mm
- board text added: "(C) critbit 05.2022"
- board text added: "+"
- board text added: "+++++"
- board text added: "-"
- board text added: "---"
- board text added: "1+|1-|GND"
- board text added: "2+|2-|GND"
- board text added: "AnalogDiscoveryCurrentDongle Rev. 2.0"
- board text added: "BNC->DIO ENA"
- board text added: "CH1 CURR/BNC"
- board text added: "CH2 CURR/BNC"
- board text added: "CH_A CLIP"
- board text added: "CH_B CLIP"
- board text added: "IO12"
- board text added: "IO13"
- board text added: "IO14"
- board text added: "IO5"
- board text added: "IO6"
- board text added: "VDC"
- board text added: "WAV1"
- board text added: "WAV2"
- board text removed: "+++"
- board text removed: "<-BNC"
- board text removed: "AnalogDiscovery CurrentDongle Rev. 1.1 (C) critbit"
- board text removed: "CURR->"
- board text removed: "G"
- board text removed: "W1"
- board text removed: "W2"

Commit message: fabrication outputs
Changed lines of the file:
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@@
     (fp_line (start 1 0.625) (end -1 0.625) (layer "F.Fab") (width 0.1))
     (fp_line (start -1 0.625) (end -1 -0.625) (layer "F.Fab") (width 0.1))
-    (pad "1" smd roundrect (at -0.9125 0) (size 1.025 1.4) (layers "F.Cu" "F.Paste" "F.Mask") (roundrect_rratio 0.243902)
+    (pad "1" smd roundrect (at -0.9125 0) (size 1.025 1.4) (layers "F.Cu" "F.Paste" "F.Mask") (roundrect_rratio 0.243902439)
       (net 36 "Net-(R18-Pad2)") (pintype "passive"))
-    (pad "2" smd roundrect (at 0.9125 0) (size 1.025 1.4) (layers "F.Cu" "F.Paste" "F.Mask") (roundrect_rratio 0.243902)
+    (pad "2" smd roundrect (at 0.9125 0) (size 1.025 1.4) (layers "F.Cu" "F.Paste" "F.Mask") (roundrect_rratio 0.243902439)
       (net 18 "Net-(JP7-Pad1)") (pintype "passive"))
     (model "${KICAD6_3DMODEL_DIR}/Resistor_SMD.3dshapes/R_0805_2012Metric.wrl"
@@
     (fp_line (start 1 0.625) (end -1 0.625) (layer "F.Fab") (width 0.1))
     (fp_line (start 1 -0.625) (end 1 0.625) (layer "F.Fab") (width 0.1))
-    (pad "1" smd roundrect (at -0.9125 0) (size 1.025 1.4) (layers "F.Cu" "F.Paste" "F.Mask") (roundrect_rratio 0.243902)
+    (pad "1" smd roundrect (at -0.9125 0) (size 1.025 1.4) (layers "F.Cu" "F.Paste" "F.Mask") (roundrect_rratio 0.243902439)
       (net 6 "VDC") (pintype "passive"))
-    (pad "2" smd roundrect (at 0.9125 0) (size 1.025 1.4) (layers "F.Cu" "F.Paste" "F.Mask") (roundrect_rratio 0.243902)
+    (pad "2" smd roundrect (at 0.9125 0) (size 1.025 1.4) (layers "F.Cu" "F.Paste" "F.Mask") (roundrect_rratio 0.243902439)
       (net 36 "Net-(R18-Pad2)") (pintype "passive"))
     (model "${KICAD6_3DMODEL_DIR}/Resistor_SMD.3dshapes/R_0805_2012Metric.wrl"
