File: ADCurrentDongle.kicad_pcb (KiCad board)
At the start: 4 copper layers, 37 x 74 mm, 56 parts, among them J1 EXT_SONDE1, J2 EXT_SONDE2, J3 Screw_Terminal_01x04, J4 Conn_01x02, J5 BRD_EXT, J6 R_EXT, J7 Conn_01x03, J8 Conn_01x03, J9 Conn_01x10, SW1 CH1_DPDT, SW2 CH2_DPDT, SW3 CURR_LP_SEL, SW4 CH1_DPDT, U1 INA186AxDDxx, U2 INA186AxDDxx, U3 MCP6004, U4 AnalogDiscovery2

Commit message: add support software package (LLM code), reference labSession repo, some cleanup
Other:
- board text added: "https://forum.digilent.com/topic/9333-analog-discovery-2-board-3d-model/"
