File: ADCurrentDongle.kicad_sch (KiCad schematic)
At the start: 54 parts, among them J1 EXT_SONDE1, J10 Conn_01x06, J2 EXT_SONDE2, J3 Screw_Terminal_01x04, J4 Conn_01x02, J5 BRD_EXT, J6 R_EXT, J7 Conn_01x03, J8 Conn_01x03, J9 Conn_01x03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

Commit message: adding new rev fabrication and stuff
Parts:
- gave numbers to parts that had none: 1
- renumbered JP7 to JP5, R7 to R6, R6 to R7, SW1 to SW2, SW2 to SW3
Changed lines of the file:
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@@
   (symbol (lib_id "Device:R_Small") (at 173.99 71.12 270) (unit 1)
     (in_bom yes) (on_board yes)
-    (property "Reference" "R7" (id 0) (at 170.18 69.85 90))
+    (property "Reference" "R6" (id 0) (at 170.18 69.85 90))
     (property "Value" "3k3" (id 1) (at 179.07 69.85 90))
     (property "Footprint" "Resistor_SMD:R_0402_1005Metric" (id 2) (at 173.99 71.12 0)
@@
   (symbol (lib_id "Device:R_Small") (at 173.99 86.36 270) (unit 1)
     (in_bom yes) (on_board yes)
-    (property "Reference" "R6" (id 0) (at 170.18 85.09 90))
+    (property "Reference" "R7" (id 0) (at 170.18 85.09 90))
     (property "Value" "330" (id 1) (at 179.07 85.09 90))
     (property "Footprint" "Resistor_SMD:R_0402_1005Metric" (id 2) (at 173.99 86.36 0)
@@
   (symbol (lib_id "Jumper:Jumper_2_Open") (at 389.89 43.18 270) (unit 1)
     (in_bom yes) (on_board yes)
-    (property "Reference" "JP7" (id 0) (at 392.3792 42.0116 90)
+    (property "Reference" "JP5" (id 0) (at 392.3792 42.0116 90)
       (effects (font (size 1.27 1.27)) (justify left))
     )
@@
   (symbol (lib_id "Switch:SW_Push_DPDT") (at 349.25 82.55 0) (mirror y) (unit 1)
     (in_bom yes) (on_board yes) (fields_autoplaced)
-    (property "Reference" "SW2" (id 0) (at 349.25 70.5825 0))
+    (property "Reference" "SW3" (id 0) (at 349.25 70.5825 0))
     (property "Value" "CH2_DPDT" (id 1) (at 349.25 73.3576 0))
     (property "Footprint" "Button_Switch_SMD:SW_DPDT_CK_JS202011JCQN" (id 2) (at 349.25 77.47 0)
@@
   (symbol (lib_id "Switch:SW_Push_DPDT") (at 185.42 93.98 0) (mirror y) (unit 1)
     (in_bom yes) (on_board yes)
-    (property "Reference" "SW?" (id 0) (at 187.96 92.71 0))
+    (property "Reference" "SW1" (id 0) (at 187.96 92.71 0))
     (property "Value" "CURR_LP_SEL" (id 1) (at 193.04 95.25 0))
     (property "Footprint" "Button_Switch_SMD:SW_DPDT_CK_JS202011JCQN" (id 2) (at 185.42 88.9 0)
@@
   (symbol (lib_id "Switch:SW_Push_DPDT") (at 347.98 49.53 0) (mirror y) (unit 1)
     (in_bom yes) (on_board yes) (fields_autoplaced)
-    (property "Reference" "SW1" (id 0) (at 347.98 37.5625 0))
+    (property "Reference" "SW2" (id 0) (at 347.98 37.5625 0))
     (property "Value" "CH1_DPDT" (id 1) (at 347.98 40.3376 0))
     (property "Footprint" "Button_Switch_SMD:SW_DPDT_CK_JS202011JCQN" (id 2) (at 347.98 44.45 0)
@@
     )
     (path "/00000000-0000-0000-0000-00006014f55c"
-      (reference "JP7") (unit 1) (value "Jumper_2_Open") (footprint "Connector_PinHeader_2.54mm:PinHeader_1x02_P2.54mm_Vertical")
+      (reference "JP5") (unit 1) (value "Jumper_2_Open") (footprint "Connector_PinHeader_2.54mm:PinHeader_1x02_P2.54mm_Vertical")
     )
     (path "/00000000-0000-0000-0000-00005fbed4cf"
@@
       (reference "R5") (unit 1) (value "100") (footprint "Resistor_SMD:R_0402_1005Metric")
     )
+    (path "/00000000-0000-0000-0000-00005fb58ac0"
+      (reference "R6") (unit 1) (value "3k3") (footprint "Resistor_SMD:R_0402_1005Metric")
+    )
     (path "/00000000-0000-0000-0000-00005fbde573"
-      (reference "R6") (unit 1) (value "330") (footprint "Resistor_SMD:R_0402_1005Metric")
-    )
-    (path "/00000000-0000-0000-0000-00005fb58ac0"
-      (reference "R7") (unit 1) (value "3k3") (footprint "Resistor_SMD:R_0402_1005Metric")
+      (reference "R7") (unit 1) (value "330") (footprint "Resistor_SMD:R_0402_1005Metric")
     )
     (path "/00000000-0000-0000-0000-00005fbde742"
@@
       (reference "R19") (unit 1) (value "50") (footprint "Resistor_SMD:R_0805_2012Metric")
     )
+    (path "/5d49d8db-07c2-4dac-b489-ffb4c77b0a1d"
+      (reference "SW1") (unit 1) (value "CURR_LP_SEL") (footprint "Button_Switch_SMD:SW_DPDT_CK_JS202011JCQN")
+    )
     (path "/7d0ebe33-f0fd-480e-8246-b968f71087af"
-      (reference "SW1") (unit 1) (value "CH1_DPDT") (footprint "Button_Switch_SMD:SW_DPDT_CK_JS202011JCQN")
+      (reference "SW2") (unit 1) (value "CH1_DPDT") (footprint "Button_Switch_SMD:SW_DPDT_CK_JS202011JCQN")
     )
     (path "/07030f91-3374-4871-b526-4680a1f088d7"
-      (reference "SW2") (unit 1) (value "CH2_DPDT") (footprint "Button_Switch_SMD:SW_DPDT_CK_JS202011JCQN")
-    )
-    (path "/5d49d8db-07c2-4dac-b489-ffb4c77b0a1d"
-      (reference "SW?") (unit 1) (value "CURR_LP_SEL") (footprint "Button_Switch_SMD:SW_DPDT_CK_JS202011JCQN")
+      (reference "SW3") (unit 1) (value "CH2_DPDT") (footprint "Button_Switch_SMD:SW_DPDT_CK_JS202011JCQN")
     )
     (path "/00000000-0000-0000-0000-00005fe5ec53"
