File: ADCurrentDongle.kicad_sch (KiCad schematic)
At the start: 54 parts, among them J1 EXT_SONDE1, J10 Conn_01x06, J2 EXT_SONDE2, J3 Screw_Terminal_01x04, J4 Conn_01x02, J5 BRD_EXT, J6 R_EXT, J7 Conn_01x03, J8 Conn_01x03, J9 Conn_01x03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

Commit message: pre order commit
Parts:
- removed J10: Conn_01x06, Connector_PinHeader_2.54mm:PinHeader_1x06_P2.54mm_Vertical, symbol Connector_Generic:Conn_01x06
- removed J9: Conn_01x03, Connector_PinHeader_2.54mm:PinHeader_1x03_P2.54mm_Vertical, symbol Connector_Generic:Conn_01x03
- added D5: LED, LED_SMD:LED_0603_1608Metric, symbol Device:LED
- added J9: (no value), symbol Connector_Generic:Conn_01x10
- added R20: 3k3, Resistor_SMD:R_0402_1005Metric, symbol Device:R_Small
- added SW4: CH1_DPDT, Button_Switch_SMD:SW_DPDT_CK_JS202011JCQN, symbol Switch:SW_Push_DPDT
- J4: footprint Connector_PinHeader_2.54mm:PinHeader_1x02_P2.54mm_Horizontal -> Connector_PinHeader_2.54mm:PinHeader_1x02_P2.54mm_Vertical
- gave numbers to parts that had none: 1
Connections:
- net GND: now also D5.1 (K), J9.1 (Pin_1), J9.10 (Pin_10)
- net VDC: now also J9.4 (Pin_4), R20.1
- net CMEAS_A: now reaches C5.1, R7.1, SW1.3 (C), SW3.2 (B), U3.3 (+)
- net CMEAS_B: now reaches C6.1, R9.1, SW2.3 (C), SW3.5 (B), U3.5 (+)
- net CH1_INP: now reaches J1.1 (In), J7.1 (Pin_1), SW1.1 (A)
- net CH1_INP: now also SW4.1 (A)
- net CH1_INM: now reaches J1.2 (Ext), J7.2 (Pin_2), SW1.4 (A)
- net CMEAS_B_CLIP: now reaches D3.2 (A), U3.8, U4.2 (DIO15)
- net CMEAS_A_CLIP: now reaches U4.1 (DIO7)
- net CMEAS_A_CLIP: now also D4.2 (A), U3.14
- net CH1_DIO: now reaches U4.15 (DIO0)
- net CH1_DIO: now also SW4.2 (B)
- net CH2_DIO: now reaches U4.16 (DIO8)
- net CH2_DIO: now also SW4.5 (B)
- net WAV_GEN1: now reaches U4.21 (WAV_GEN1)
- net WAV_GEN1: now also J9.2 (Pin_2)
- net WAV_GEN2: now reaches U4.22 (WAV_GEN2)
- net WAV_GEN2: now also J9.3 (Pin_3)
- net DIO6: now reaches U4.3 (DIO6)
- net DIO6: now also J9.9 (Pin_9)
- net DIO5: now reaches U4.5 (DIO5)
- net DIO5: now also J9.7 (Pin_7)
- net DIO13: now reaches U4.6 (DIO13)
- net DIO13: now also J9.6 (Pin_6)
- net DIO12: now reaches U4.8 (DIO12)
- net DIO12: now also J9.5 (Pin_5)
- net CH2_INP: now reaches J2.1 (In), J8.1 (Pin_1), SW2.1 (A)
- net CH2_INP: now also SW4.4 (A)
- net CH2_INM: now reaches J2.2 (Ext), J8.2 (Pin_2), SW2.4 (A)
- new net: D5.2 (A), R20.2
- new net DIO14: J9.8 (Pin_8), U4.4 (DIO14)
- no-connect marks 15 -> 9
Other:
- note added: "Without those sinking resistors, supply output gets very noisy"
- note removed: "Without this, supply is very noisy"
- moved on the sheet: C1, C2, C3, C4, C5, C6, C7, C8, C9, D1, D2, D3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

Commit message: fabrication outputs
Parts:
- J9: value (none) -> Conn_01x10; footprint (none) -> Connector_PinHeader_2.54mm:PinHeader_1x10_P2.54mm_Vertical
Changed lines of the file:
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@@
     (in_bom yes) (on_board yes) (fields_autoplaced)
     (property "Reference" "J9" (id 0) (at 287.02 196.9602 0))
-    (property "Value" "" (id 1) (at 287.02 199.4971 0))
-    (property "Footprint" "" (id 2) (at 287.02 212.09 0)
+    (property "Value" "Conn_01x10" (id 1) (at 287.02 199.4971 0))
+    (property "Footprint" "Connector_PinHeader_2.54mm:PinHeader_1x10_P2.54mm_Vertical" (id 2) (at 287.02 212.09 0)
       (effects (font (size 1.27 1.27)) hide)
     )
